File: stm32l432kcu6_eval/stm32l432kcu6_eval.kicad_pcb (KiCad board)
At the start: 2 copper layers, 19 parts, among them J1 Conn_01x04_Pin, J2 Conn_01x04_Pin, J3 USB_C_Receptacle, U1 STM32L432KCUx, U2 XC6206PxxxMR, U3 USBLC6-2SC6, Y1 ASFL1-40.000MHZ-EC-T, Y2 FC-135_32.7680KA-A3

Commit message: board save 4
Parts:
- removed C4: C_Small, Capacitor_SMD:C_0603_1608Metric
- added C10: 100nF, Capacitor_SMD:C_0603_1608Metric, F.Cu at (194.8, 89.0)
- added C11: 100nF, Capacitor_SMD:C_0603_1608Metric, F.Cu at (194.8, 91.5)
- added J4: Conn_01x20_Pin, Connector_PinSocket_2.54mm:PinSocket_1x20_P2.54mm_Vertical, F.Cu at (134.0, 75.5)
- added R1: 10K, Resistor_SMD:R_0603_1608Metric, F.Cu at (194.8, 94.0)
- added S1: B3U-1000PM, custom_part_library_1:B3U1000PM_3D_MODEL, F.Cu at (199.4, 89.6)
- added S2: B3U-1000PM, custom_part_library_1:B3U1000PM_3D_MODEL, F.Cu at (199.4, 93.3)
- C3, C5, C6: value C_Small -> 100nF
- FB1: value FerriteBead_Small -> value
- J2: value Conn_01x04_Pin -> Conn_01x20_Pin; footprint Connector_PinSocket_2.54mm:PinSocket_1x04_P2.54mm_Horizontal -> Connector_PinSocket_2.54mm:PinSocket_1x20_P2.54mm_Vertical
- Y2: value FC-135_32.7680KA-A3 -> FC-135_32.7680KA-A3_12_5_pF; footprint FC_135_CLOCK_KI_CAD:FC135327680KAA3 -> FC_135_CLOCK_KI_CAD:FC-135_32_7680KA-A3
- moved J3 46.0 mm to (151.0, 127.0)
- moved C2 45.4 mm to (195.0, 123.0)
- moved C1 44.0 mm to (195.0, 117.0)
- moved J2 36.7 mm to (164.0, 124.1), turned to 180 degrees
- moved C8 35.5 mm to (176.0, 141.0)
- moved C6 35.5 mm to (176.0, 136.0)
- moved C7 35.5 mm to (176.0, 138.5)
- moved C9 35.5 mm to (176.0, 143.5)
- moved C3 32.2 mm to (147.0, 118.0), turned to 90 degrees
- moved U2 31.5 mm to (144.0, 119.0)
- moved C5 31.2 mm to (188.4, 79.4)
- moved F1 31.2 mm to (188.4, 81.9)
- moved FB1 31.2 mm to (188.4, 84.4)
- moved U3 20.4 mm to (151.1, 114.1), turned to 90 degrees
- moved Y2 17.4 mm to (143.0, 105.0), turned to -45 degrees
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Connections:
- C1 pad 1: unconnected-(C1-Pad1) -> /mcu_osccillators/PC15(OSC_OUT)
- C1 pad 2: unconnected-(C1-Pad2) -> GND
- C2 pad 1: unconnected-(C2-Pad1) -> /mcu_osccillators/PC14(OSC_IN)
- C2 pad 2: unconnected-(C2-Pad2) -> GND
- C3 pad 1: unconnected-(C3-Pad1) -> Net-(U2-VI)
- C3 pad 2: unconnected-(C3-Pad2) -> GND
- C5 pad 1: unconnected-(C5-Pad1) -> +3V3
- C5 pad 2: unconnected-(C5-Pad2) -> GND
- C7 pad 1: Net-(U1-VDDA) -> +3V3
- C8 pad 1: Net-(U1-VDDA) -> +3V3
- C9 pad 1: Net-(U1-VDDA) -> +3V3
- F1 pad 1: unconnected-(F1-Pad1) -> +5V_USB
- F1 pad 2: unconnected-(F1-Pad2) -> Net-(F1-Pad2)
- FB1 pad 1: unconnected-(FB1-Pad1) -> Net-(F1-Pad2)
- FB1 pad 2: unconnected-(FB1-Pad2) -> Net-(U2-VI)
- J1 pad 1: /connectors_gpios_2_5_4/test_3 -> +3V3
- J1 pad 2: unconnected-(J1-Pin_2-Pad2) -> /connectors_gpios_2_5_4/PA13
- J1 pad 3: unconnected-(J1-Pin_3-Pad3) -> /connectors_gpios_2_5_4/PA14
- J1 pad 4: unconnected-(J1-Pin_4-Pad4) -> GND
- J2 pad 1: unconnected-(J2-Pin_1-Pad1) -> /connectors_gpios_2_5_4/PA0
- J2 pad 2: unconnected-(J2-Pin_2-Pad2) -> /connectors_gpios_2_5_4/PA1
- J2 pad 3: unconnected-(J2-Pin_3-Pad3) -> /connectors_gpios_2_5_4/PA2
- J2 pad 4: unconnected-(J2-Pin_4-Pad4) -> /connectors_gpios_2_5_4/PA3
- J3 pad A1: Net-(J3-GND-PadA1) -> GND
- J3 pad A12: Net-(J3-GND-PadA1) -> GND
- J3 pad A4: Net-(J3-VBUS-PadA4) -> +5V_USB
- J3 pad A6: unconnected-(J3-D+-PadA6) -> USB_D+
- J3 pad A7: unconnected-(J3-D--PadA7) -> USB_D-
- J3 pad A9: Net-(J3-VBUS-PadA4) -> +5V_USB
- J3 pad B1: Net-(J3-GND-PadA1) -> GND
- J3 pad B12: Net-(J3-GND-PadA1) -> GND
- J3 pad B4: Net-(J3-VBUS-PadA4) -> +5V_USB
- J3 pad B6: unconnected-(J3-D+-PadB6) -> USB_D+
- J3 pad B7: unconnected-(J3-D--PadB7) -> USB_D-
- J3 pad B9: Net-(J3-VBUS-PadA4) -> +5V_USB
- J3 pad S1: unconnected-(J3-SHIELD-PadS1) -> GND
- U1 pad 1: Net-(U1-VDDA) -> +3V3
- U1 pad 10: unconnected-(U1-PA4-Pad10) -> /connectors_gpios_2_5_4/PA4
- U1 pad 11: unconnected-(U1-PA5-Pad11) -> /connectors_gpios_2_5_4/PA5
- U1 pad 12: unconnected-(U1-PA6-Pad12) -> /connectors_gpios_2_5_4/PA6
- U1 pad 13: unconnected-(U1-PA7-Pad13) -> /connectors_gpios_2_5_4/PA7
- U1 pad 14: unconnected-(U1-PB0-Pad14) -> /mcu_osccillators/PB0
- U1 pad 15: unconnected-(U1-PB1-Pad15) -> /mcu_osccillators/PB1
- U1 pad 16: Net-(U1-VSS-Pad16) -> GND
- U1 pad 17: Net-(U1-VDDA) -> +3V3
- U1 pad 18: unconnected-(U1-PA8-Pad18) -> /connectors_gpios_2_5_4/PA8
- U1 pad 19: unconnected-(U1-PA9-Pad19) -> /connectors_gpios_2_5_4/PA9
- U1 pad 2: unconnected-(U1-PC14-Pad2) -> /mcu_osccillators/PC14(OSC_IN)
- U1 pad 20: unconnected-(U1-PA10-Pad20) -> /connectors_gpios_2_5_4/PA10
- U1 pad 21: unconnected-(U1-PA11-Pad21) -> /connectors_gpios_2_5_4/PA11
- U1 pad 22: unconnected-(U1-PA12-Pad22) -> /connectors_gpios_2_5_4/PA12
- U1 pad 23: unconnected-(U1-PA13-Pad23) -> /connectors_gpios_2_5_4/PA13
- U1 pad 24: unconnected-(U1-PA14-Pad24) -> /connectors_gpios_2_5_4/PA14
- U1 pad 25: unconnected-(U1-PA15-Pad25) -> /connectors_gpios_2_5_4/PA15
- U1 pad 26: unconnected-(U1-PB3-Pad26) -> /mcu_osccillators/PB3
- U1 pad 27: unconnected-(U1-PB4-Pad27) -> /mcu_osccillators/PB4
- U1 pad 28: unconnected-(U1-PB5-Pad28) -> /mcu_osccillators/PB5
- U1 pad 29: unconnected-(U1-PB6-Pad29) -> /mcu_osccillators/PB6
- U1 pad 3: unconnected-(U1-PC15-Pad3) -> /mcu_osccillators/PC15(OSC_OUT)
- U1 pad 30: unconnected-(U1-PB7-Pad30) -> /mcu_osccillators/PB7
- U1 pad 31: unconnected-(U1-PH3-Pad31) -> /mcu_osccillators/PH3(BOOT)
- U1 pad 32: Net-(U1-VSS-Pad16) -> GND
- U1 pad 33: Net-(U1-VSS-Pad16) -> GND
- U1 pad 4: unconnected-(U1-NRST-Pad4) -> /mcu_osccillators/NRST
- U1 pad 5: Net-(U1-VDDA) -> +3V3
- U1 pad 6: unconnected-(U1-PA0-Pad6) -> /connectors_gpios_2_5_4/PA0
- U1 pad 7: unconnected-(U1-PA1-Pad7) -> /connectors_gpios_2_5_4/PA1
- U1 pad 8: /mcu_osccillators/test_1 -> /connectors_gpios_2_5_4/PA2
- U1 pad 9: /connectors_gpios_2_5_4/test_3 -> /connectors_gpios_2_5_4/PA3
- U2 pad 1: unconnected-(U2-GND-Pad1) -> GND
- U2 pad 2: unconnected-(U2-VO-Pad2) -> +3V3
- U2 pad 3: unconnected-(U2-VI-Pad3) -> Net-(U2-VI)
- U3 pad 1: unconnected-(U3-I/O1-Pad1) -> USB_D+
- U3 pad 2: unconnected-(U3-GND-Pad2) -> GND
- U3 pad 3: unconnected-(U3-I/O2-Pad3) -> USB_D-
- U3 pad 4: unconnected-(U3-I/O2-Pad4) -> /power_usb/MCU_USB_DM
- U3 pad 5: unconnected-(U3-VBUS-Pad5) -> +5V_USB
- U3 pad 6: unconnected-(U3-I/O1-Pad6) -> /power_usb/MCU_USB_DP
- Y1 pad 3: unconnected-(Y1-OUTPUT-Pad3) -> /connectors_gpios_2_5_4/PA0
- Y2 pad 1: unconnected-(Y2-Pad1) -> /mcu_osccillators/PC14(OSC_IN)
- Y2 pad 2: unconnected-(Y2-X2-Pad2) -> /mcu_osccillators/PC15(OSC_OUT)

Commit message: pin arragment 1
Parts:
- removed J3: USB_C_Receptacle, Connector_USB:USB_C_Receptacle_Molex_105450-0101
- added C4: 100nF, Capacitor_SMD:C_0603_1608Metric, F.Cu at (170.9, 110.8)
- added D1: LED, LED_SMD:LED_0603_1608Metric, F.Cu at (199.2, 103.0)
- added D2: LED, LED_SMD:LED_0603_1608Metric, F.Cu at (157.1, 136.2)
- added J5: USB_B_Micro, Connector_USB:USB_Micro-B_Molex-105017-0001, F.Cu at (150.0, 122.9)
- added R2: R_Small, Resistor_SMD:R_0603_1608Metric, F.Cu at (195.2, 105.5)
- added R3: R_Small, Resistor_SMD:R_0603_1608Metric, F.Cu at (153.1, 136.2)
- added R4: R_Small, Resistor_SMD:R_0603_1608Metric, F.Cu at (153.1, 138.7)
- added R5: R_Small, Resistor_SMD:R_0603_1608Metric, F.Cu at (153.1, 141.2)
- added R6: R_Small, Resistor_SMD:R_0603_1608Metric, F.Cu at (195.6, 95.9)
- added S3: B3U-1000PM, custom_part_library_1:B3U1000PM_3D_MODEL, F.Cu at (168.7, 110.8)
- moved S1 67.0 mm to (132.5, 93.7), turned to 45 degrees
- moved J4 55.8 mm to (161.4, 124.1), turned to 180 degrees
- moved F1 55.4 mm to (144.8, 116.0), turned to 180 degrees
- moved J2 54.5 mm to (138.6, 75.9), turned to 0 degrees
- moved FB1 53.0 mm to (144.8, 114.5)
- moved S2 29.8 mm to (169.6, 92.8), turned to 135 degrees
- moved Y1 19.6 mm to (126.7, 111.9)
- moved Y2 13.5 mm to (129.6, 103.3)
- moved R1 13.4 mm to (185.1, 103.3)
- moved U2 9.10 mm to (144.2, 109.9)
- moved C3 5.46 mm to (144.8, 113.0), turned to 180 degrees
- moved U3 3.64 mm to (149.7, 117.5)
- moved J1 2.62 mm to (153.8, 84.1)
Connections:
- C1 pad 1: /mcu_osccillators/PC15(OSC_OUT) -> /connectors_gpios_2_5_4/PC15(OSC_OUT)
- C10 pad 1: /mcu_osccillators/NRST -> /connectors_gpios_2_5_4/NRST
- C11 pad 1: /mcu_osccillators/PH3(BOOT) -> Net-(C11-Pad1)
- C2 pad 1: /mcu_osccillators/PC14(OSC_IN) -> /connectors_gpios_2_5_4/PC14(OSC_IN)
- J2 pad 1: /connectors_gpios_2_5_4/PA0 -> unconnected-(J2-Pin_1-Pad1)
- J2 pad 10: /connectors_gpios_2_5_4/PA9 -> /connectors_gpios_2_5_4/PH3(BOOT)
- J2 pad 11: /connectors_gpios_2_5_4/PA10 -> /connectors_gpios_2_5_4/PC14(OSC_IN)
- J2 pad 12: /connectors_gpios_2_5_4/PA11 -> /connectors_gpios_2_5_4/PC15(OSC_OUT)
- J2 pad 13: /connectors_gpios_2_5_4/PA12 -> /connectors_gpios_2_5_4/NRST
- J2 pad 14: /connectors_gpios_2_5_4/PA13 -> /connectors_gpios_2_5_4/PA0
- J2 pad 15: /connectors_gpios_2_5_4/PA14 -> /connectors_gpios_2_5_4/PA1
- J2 pad 16: /connectors_gpios_2_5_4/PA15 -> /connectors_gpios_2_5_4/PA2
- J2 pad 2: /connectors_gpios_2_5_4/PA1 -> unconnected-(J2-Pin_2-Pad2)
- J2 pad 3: /connectors_gpios_2_5_4/PA2 -> unconnected-(J2-Pin_3-Pad3)
- J2 pad 4: /connectors_gpios_2_5_4/PA3 -> /connectors_gpios_2_5_4/PA15
- J2 pad 5: /connectors_gpios_2_5_4/PA4 -> /connectors_gpios_2_5_4/PB3
- J2 pad 6: /connectors_gpios_2_5_4/PA5 -> /connectors_gpios_2_5_4/PB4
- J2 pad 7: /connectors_gpios_2_5_4/PA6 -> /connectors_gpios_2_5_4/PB5
- J2 pad 8: /connectors_gpios_2_5_4/PA7 -> /connectors_gpios_2_5_4/PB6
- J2 pad 9: /connectors_gpios_2_5_4/PA8 -> /connectors_gpios_2_5_4/PB7
- J4 pad 1: /connectors_gpios_2_5_4/PB0 -> unconnected-(J4-Pin_1-Pad1)
- J4 pad 10: /connectors_gpios_2_5_4/PC14(OSC_IN) -> /connectors_gpios_2_5_4/PA7
- J4 pad 11: /connectors_gpios_2_5_4/PC14(OSC_IN) -> /connectors_gpios_2_5_4/PA8
- J4 pad 12: unconnected-(J4-Pin_12-Pad12) -> /connectors_gpios_2_5_4/PA9
- J4 pad 13: unconnected-(J4-Pin_13-Pad13) -> /connectors_gpios_2_5_4/PA10
- J4 pad 14: unconnected-(J4-Pin_14-Pad14) -> /connectors_gpios_2_5_4/PA11
- J4 pad 15: unconnected-(J4-Pin_15-Pad15) -> /connectors_gpios_2_5_4/PA12
- J4 pad 16: unconnected-(J4-Pin_16-Pad16) -> /connectors_gpios_2_5_4/PA13
- J4 pad 17: unconnected-(J4-Pin_17-Pad17) -> /connectors_gpios_2_5_4/PA14
- J4 pad 2: /connectors_gpios_2_5_4/PB1 -> unconnected-(J4-Pin_2-Pad2)
- J4 pad 3: /connectors_gpios_2_5_4/PB3 -> unconnected-(J4-Pin_3-Pad3)
- J4 pad 4: /connectors_gpios_2_5_4/PB4 -> unconnected-(J4-Pin_4-Pad4)
- J4 pad 5: /connectors_gpios_2_5_4/PB5 -> unconnected-(J4-Pin_5-Pad5)
- J4 pad 6: /connectors_gpios_2_5_4/PB6 -> /connectors_gpios_2_5_4/PA3
- J4 pad 7: /connectors_gpios_2_5_4/PB7 -> /connectors_gpios_2_5_4/PA4
- J4 pad 8: /connectors_gpios_2_5_4/NRST -> /connectors_gpios_2_5_4/PA5
- J4 pad 9: /connectors_gpios_2_5_4/PH3(BOOT) -> /connectors_gpios_2_5_4/PA6
- R1 pad 1: /mcu_osccillators/PH3(BOOT) -> /connectors_gpios_2_5_4/PH3(BOOT0)
- S1 pad 1: +3V3 -> GND
- S1 pad 2: /mcu_osccillators/PH3(BOOT) -> /connectors_gpios_2_5_4/NRST
- S2 pad 1: GND -> +3V3
- S2 pad 2: /mcu_osccillators/NRST -> /connectors_gpios_2_5_4/PH3(BOOT0)
- U1 pad 14: /mcu_osccillators/PB0 -> /connectors_gpios_2_5_4/PB0
- U1 pad 15: /mcu_osccillators/PB1 -> /connectors_gpios_2_5_4/PB1
- U1 pad 2: /mcu_osccillators/PC14(OSC_IN) -> /connectors_gpios_2_5_4/PC14(OSC_IN)
- U1 pad 26: /mcu_osccillators/PB3 -> /connectors_gpios_2_5_4/PB3
- U1 pad 27: /mcu_osccillators/PB4 -> /connectors_gpios_2_5_4/PB4
- U1 pad 28: /mcu_osccillators/PB5 -> /connectors_gpios_2_5_4/PB5
- U1 pad 29: /mcu_osccillators/PB6 -> /connectors_gpios_2_5_4/PB6
- U1 pad 3: /mcu_osccillators/PC15(OSC_OUT) -> /connectors_gpios_2_5_4/PC15(OSC_OUT)
- U1 pad 30: /mcu_osccillators/PB7 -> /connectors_gpios_2_5_4/PB7
- U1 pad 31: /mcu_osccillators/PH3(BOOT) -> /connectors_gpios_2_5_4/PH3(BOOT)
- U1 pad 4: /mcu_osccillators/NRST -> /connectors_gpios_2_5_4/NRST
- U3 pad 1: USB_D+ -> /power_usb/USB_M+
- U3 pad 3: USB_D- -> /power_usb/USB_M-
- U3 pad 4: /power_usb/MCU_USB_DM -> /connectors_gpios_2_5_4/PA11
- U3 pad 6: /power_usb/MCU_USB_DP -> /connectors_gpios_2_5_4/PA12
- Y2 pad 1: /mcu_osccillators/PC14(OSC_IN) -> /connectors_gpios_2_5_4/PC14(OSC_IN)
- Y2 pad 2: /mcu_osccillators/PC15(OSC_OUT) -> /connectors_gpios_2_5_4/PC15(OSC_OUT)
Routing:
- net /connectors_gpios_2_5_4/PA12: track 0.00 -> 19.1 mm
- net /connectors_gpios_2_5_4/PA11: track 0.00 -> 16.0 mm
- net /connectors_gpios_2_5_4/PA13: track 0.00 -> 13.7 mm
- net /connectors_gpios_2_5_4/PA14: track 0.00 -> 13.7 mm
- net +5V_USB: track 0.00 -> 11.2 mm
- net /power_usb/USB_M-: track 0.00 -> 3.46 mm
- net /power_usb/USB_M+: track 0.00 -> 3.44 mm
- net /connectors_gpios_2_5_4/PA6: track 0.00 -> 3.00 mm, vias 0 -> 1
- net /connectors_gpios_2_5_4/PA7: track 0.00 -> 2.98 mm, vias 0 -> 1
- net /connectors_gpios_2_5_4/PA10: track 0.00 -> 2.78 mm, vias 0 -> 1
- net /connectors_gpios_2_5_4/PA4: track 0.00 -> 2.30 mm, vias 0 -> 1
- net /connectors_gpios_2_5_4/PA5: track 0.00 -> 1.80 mm, vias 0 -> 1
- net /connectors_gpios_2_5_4/PB0: track 0.00 -> 1.78 mm, vias 0 -> 1
- net /connectors_gpios_2_5_4/PA3: track 0.00 -> 1.68 mm, vias 0 -> 1
- net /connectors_gpios_2_5_4/PA8: track 0.00 -> 1.55 mm, vias 0 -> 1
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Other:
- board outline added: 27.4 x 53 mm
- copper layers 2 -> 4
