File: stm32l432kcu6_eval/stm32l432kcu6_eval.kicad_pcb (KiCad board)
At the start: 4 copper layers, 27.4 x 53 mm, 33 parts, among them J1 Conn_01x04_Pin, J2 Conn_01x20_Pin, J4 Conn_01x20_Pin, J5 USB_B_Micro, U1 STM32L432KCUx, U2 XC6206PxxxMR, U3 USBLC6-2SC6, Y1 ASFL1-40.000MHZ-EC-T, Y2 FC-135_32.7680KA-A3_12_5_pF

Commit message: organisation save 2
Parts:
- removed J5: USB_B_Micro, Connector_USB:USB_Micro-B_Molex-105017-0001
- added J3: Conn_01x20_Pin, Connector_PinHeader_2.54mm:PinHeader_1x20_P2.54mm_Vertical, F.Cu at (161.4, 124.1)
- C1, C2: value C_Small -> 100nF; footprint Capacitor_SMD:C_0402_1005Metric -> Capacitor_SMD:C_0603_1608Metric
- C4, C5: value 100nF -> 20pF; footprint Capacitor_SMD:C_0603_1608Metric -> Capacitor_SMD:C_0402_1005Metric
- C6: value 100nF -> 4.7uF
- C7: value C_Small -> 1uF
- C8, C9: value C_Small -> 100nF
- J1: value Conn_01x04_Pin -> USB_B_Micro; footprint Connector_PinHeader_2.54mm:PinHeader_1x04_P2.54mm_Horizontal -> Connector_USB:USB_Micro-B_Molex-105017-0001
- J4: value Conn_01x20_Pin -> Conn_01x04_Pin; footprint Connector_PinHeader_2.54mm:PinHeader_1x20_P2.54mm_Vertical -> Connector_PinHeader_2.54mm:PinHeader_1x04_P2.54mm_Horizontal
- R1: value 10K -> 0ohm
- R2, R4: value R_Small -> 1K
- R3, R6: value R_Small -> 0ohm
- R5: value R_Small -> 10K
- U1: value STM32L432KCUx -> USBLC6-2SC6; footprint Package_DFN_QFN:QFN-32-1EP_5x5mm_P0.5mm_EP3.65x3.65mm_ThermalVias -> Package_TO_SOT_SMD:SOT-23-6
- U3: value USBLC6-2SC6 -> STM32L432KCUx; footprint Package_TO_SOT_SMD:SOT-23-6 -> Package_DFN_QFN:QFN-32-1EP_5x5mm_P0.5mm_EP3.65x3.65mm_ThermalVias
- moved C5 46.2 mm to (142.5, 103.4), turned to -135 degrees
- moved J4 40.7 mm to (153.8, 84.1), turned to 90 degrees
- moved J1 39.0 mm to (150.0, 122.9), turned to 0 degrees
- moved C4 32.0 mm to (144.3, 105.1), turned to -135 degrees
- moved R4 28.1 mm to (152.7, 90.9)
- moved C11 24.3 mm to (173.7, 112.7)
- moved R1 23.2 mm to (156.8, 118.7), turned to 90 degrees
- moved R6 18.5 mm to (173.9, 114.7)
- moved C6 18.2 mm to (129.5, 98.3), turned to 45 degrees
- moved U1 17.5 mm to (149.7, 117.5), turned to -90 degrees
- moved U3 17.5 mm to (150.0, 100.0), turned to 45 degrees
- moved R5 14.7 mm to (167.2, 87.6)
- moved C1 12.3 mm to (143.4, 118.1), turned to 180 degrees
- moved C10 11.7 mm to (186.8, 97.5)
- moved C8 10.5 mm to (148.7, 137.2)
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Connections:
- C1 pad 1: /connectors_gpios_2_5_4/PC15(OSC_OUT) -> Net-(U2-VI)
- C10 pad 1: /connectors_gpios_2_5_4/NRST -> /connectors_gpios_2_5_4/PH3(BOOT0)
- C2 pad 1: /connectors_gpios_2_5_4/PC14(OSC_IN) -> +3V3
- C3 pad 1: Net-(U2-VI) -> +3V3
- C4 pad 1: /connectors_gpios_2_5_4/PH3(BOOT0) -> /connectors_gpios_2_5_4/PC15(OSC_OUT)
- C5 pad 1: +3V3 -> /connectors_gpios_2_5_4/PC14(OSC_IN)
- C9 pad 1: +3V3 -> /connectors_gpios_2_5_4/NRST
- J1 pad 1: GND -> +5V_USB
- J1 pad 2: /connectors_gpios_2_5_4/PA14 -> /power_usb/USB_M-
- J1 pad 3: /connectors_gpios_2_5_4/PA13 -> /power_usb/USB_M+
- J1 pad 4: +3V3 -> unconnected-(J1-ID-Pad4)
- J4 pad 1: unconnected-(J4-Pin_1-Pad1) -> GND
- J4 pad 2: unconnected-(J4-Pin_2-Pad2) -> /connectors_gpios_2_5_4/PA14
- J4 pad 3: unconnected-(J4-Pin_3-Pad3) -> /connectors_gpios_2_5_4/PA13
- J4 pad 4: /connectors_gpios_2_5_4/PA3 -> +3V3
- R1 pad 1: /connectors_gpios_2_5_4/PH3(BOOT0) -> +3V3
- R1 pad 2: GND -> Net-(R1-Pad2)
- R2 pad 1: Net-(R2-Pad1) -> Net-(R1-Pad2)
- R3 pad 1: Net-(R3-Pad1) -> /connectors_gpios_2_5_4/PB1
- R3 pad 2: Net-(D2-A) -> Net-(R3-Pad2)
- R4 pad 1: +3V3 -> Net-(R3-Pad2)
- R4 pad 2: Net-(R2-Pad1) -> Net-(D2-A)
- R5 pad 1: /connectors_gpios_2_5_4/PB1 -> /connectors_gpios_2_5_4/PH3(BOOT0)
- R5 pad 2: Net-(R3-Pad1) -> GND
- U1 pad 1: +3V3 -> /connectors_gpios_2_5_4/PA12
- U1 pad 2: /connectors_gpios_2_5_4/PC14(OSC_IN) -> GND
- U1 pad 3: /connectors_gpios_2_5_4/PC15(OSC_OUT) -> /connectors_gpios_2_5_4/PA11
- U1 pad 4: /connectors_gpios_2_5_4/NRST -> /power_usb/USB_M-
- U1 pad 5: +3V3 -> +5V_USB
- U1 pad 6: /connectors_gpios_2_5_4/PA0 -> /power_usb/USB_M+
- U3 pad 1: /power_usb/USB_M+ -> +3V3
- U3 pad 2: GND -> /connectors_gpios_2_5_4/PC14(OSC_IN)
- U3 pad 3: /power_usb/USB_M- -> /connectors_gpios_2_5_4/PC15(OSC_OUT)
- U3 pad 4: /connectors_gpios_2_5_4/PA11 -> /connectors_gpios_2_5_4/NRST
- U3 pad 5: +5V_USB -> +3V3
- U3 pad 6: /connectors_gpios_2_5_4/PA12 -> /connectors_gpios_2_5_4/PA0
Routing:
- net /connectors_gpios_2_5_4/PA2: track 0.00 -> 18.6 mm, vias 0 -> 1
- net /connectors_gpios_2_5_4/PA1: track 0.00 -> 15.2 mm, vias 0 -> 1
- net /connectors_gpios_2_5_4/PA0: track 5.33 -> 15.2 mm
- net /connectors_gpios_2_5_4/PC14(OSC_IN): track 6.34 -> 1.51 mm
- net /connectors_gpios_2_5_4/PC15(OSC_OUT): track 5.92 -> 1.45 mm
- net +3V3: track 13.8 -> 10.7 mm
- net GND: track 21.3 -> 18.6 mm, vias 11 -> 9
- net +5V_USB: track 9.71 -> 7.29 mm
- net Net-(R3-Pad2): track 0.00 -> 1.35 mm
- net Net-(R3-Pad1): track 1.35 -> 0.00 mm
- net Net-(R2-Pad1): track 1.35 -> 0.00 mm
- net Net-(R1-Pad2): track 0.00 -> 1.35 mm
- net Net-(U2-VI): track 4.88 -> 3.81 mm
- net /connectors_gpios_2_5_4/PB1: track 17.4 -> 16.4 mm
- net /connectors_gpios_2_5_4/PA12: track 27.1 -> 26.3 mm
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
Commit message: project final works save 1
Parts:
- moved C9 44.0 mm to (143.5, 93.0)
- moved C10 38.8 mm to (148.1, 94.5)
- moved C7 34.3 mm to (143.1, 99.4), turned to 45 degrees
- moved S2 22.6 mm to (147.3, 89.1), turned to 90 degrees
- moved R5 19.8 mm to (148.1, 93.0), turned to 0 degrees
- moved R3 19.3 mm to (157.7, 75.3), turned to 180 degrees
- moved R6 18.7 mm to (155.8, 110.1)
- moved C11 17.9 mm to (155.8, 111.6), turned to 180 degrees
- moved S1 17.8 mm to (142.7, 89.1), turned to 90 degrees
- moved C6 15.6 mm to (145.1, 99.4)
- moved R4 15.0 mm to (157.7, 76.8), turned to 0 degrees
- moved S3 13.1 mm to (156.6, 115.5), turned to -90 degrees
- moved D2 10.8 mm to (157.7, 78.3), turned to 0 degrees
- moved D1 7.88 mm to (156.9, 120.6), turned to 0 degrees
- moved R2 6.40 mm to (156.9, 122.1), turned to 0 degrees
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Connections:
- J2 pad 10: /connectors_gpios_2_5_4/PH3(BOOT) -> /connectors_gpios_2_5_4/PH3(BOOT0)
- J4 pad 2: /connectors_gpios_2_5_4/PA14 -> /connectors_gpios_2_5_4/PA13
- J4 pad 3: /connectors_gpios_2_5_4/PA13 -> /connectors_gpios_2_5_4/PA14
Routing:
- net /connectors_gpios_2_5_4/PB1: track 16.4 -> 39.2 mm
- net /connectors_gpios_2_5_4/PA14: track 13.7 -> 30.6 mm, vias 0 -> 2
- net GND: track 18.6 -> 33.8 mm, vias 9 -> 17
- net /connectors_gpios_2_5_4/NRST: track 12.5 -> 27.6 mm, vias 1 -> 2
- net /connectors_gpios_2_5_4/PH3(BOOT0): track 0.00 -> 15.0 mm, vias 0 -> 1
- net /connectors_gpios_2_5_4/PA13: track 13.9 -> 27.9 mm
- net /connectors_gpios_2_5_4/PA12: track 26.3 -> 40.2 mm, vias 0 -> 2
- net /connectors_gpios_2_5_4/PA11: track 25.7 -> 37.7 mm, vias 0 -> 2
- net /connectors_gpios_2_5_4/PC15(OSC_OUT): track 1.45 -> 11.9 mm
- net /connectors_gpios_2_5_4/PA1: track 15.2 -> 25.0 mm, vias 1 -> 3
- net /connectors_gpios_2_5_4/PH3(BOOT): track 8.96 -> 0.00 mm
- net /connectors_gpios_2_5_4/PC14(OSC_IN): track 1.51 -> 10.4 mm
- net +3V3: track 10.7 -> 17.1 mm, vias 6 -> 7
- net +5V_USB: track 7.29 -> 11.1 mm
- net Net-(C11-Pad1): track 0.00 -> 3.67 mm
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- added copper zone on In2.Cu, net +3V3
- added copper zone on B.Cu, net GND
- added copper zone on F.Cu, net GND
- added copper zone on In1.Cu, net GND

Commit message: project final works save 2
Parts:
- J3: moved to B.Cu
- moved C8 38.6 mm to (141.1, 99.4), turned to 45 degrees
- moved D2 12.7 mm to (153.0, 90.1)
- moved R3 12.7 mm to (153.0, 87.1)
- moved R4 12.7 mm to (153.0, 88.6)
- moved D1 1.22 mm to (156.1, 119.7)
- moved R1 1.22 mm to (156.1, 122.7)
- moved R2 1.22 mm to (156.1, 121.2)
- moved F1 0.58 mm to (144.0, 121.1)
- moved C1 0.57 mm to (144.0, 118.1)
- moved FB1 0.57 mm to (144.0, 119.6)
- turned J3 to 0 degrees
Connections:
- J2 pad 1: unconnected-(J2-Pin_1-Pad1) -> +3V3
- J2 pad 17: unconnected-(J2-Pin_17-Pad17) -> GND
- J2 pad 18: unconnected-(J2-Pin_18-Pad18) -> +3V3
- J2 pad 19: unconnected-(J2-Pin_19-Pad19) -> +5V_USB
- J2 pad 2: unconnected-(J2-Pin_2-Pad2) -> +3V3
- J2 pad 20: unconnected-(J2-Pin_20-Pad20) -> +5V_USB
- J2 pad 3: unconnected-(J2-Pin_3-Pad3) -> GND
- J3 pad 1: unconnected-(J3-Pin_1-Pad1) -> +3V3
- J3 pad 18: unconnected-(J3-Pin_18-Pad18) -> GND
- J3 pad 19: unconnected-(J3-Pin_19-Pad19) -> GND
- J3 pad 2: unconnected-(J3-Pin_2-Pad2) -> GND
- J3 pad 20: unconnected-(J3-Pin_20-Pad20) -> +3V3
- J3 pad 3: unconnected-(J3-Pin_3-Pad3) -> GND
Routing:
- net +5V_USB: track 11.1 -> 21.6 mm
- net GND: track 33.8 -> 35.2 mm
- net +3V3: track 17.1 -> 17.9 mm
Other:
- board text added: "3V3"
- board text added: "GND"
- board text added: "PA10"
- board text added: "PA11"
- board text added: "PA3"
- board text added: "PA4"
- board text added: "PA5"
- board text added: "PA6"
- board text added: "PA7"
- board text added: "PA8"
- board text added: "PA9"
- board text added: "PB1"

Commit message: project final works save 3
Parts:
- J4: moved to F.Cu
- moved J4 7.62 mm to (146.2, 84.1)
- moved J1 0.90 mm to (150.0, 123.8)
Connections:
- J4 pad 2: /connectors_gpios_2_5_4/PA13 -> /connectors_gpios_2_5_4/PA14
- J4 pad 3: /connectors_gpios_2_5_4/PA14 -> /connectors_gpios_2_5_4/PA13
Routing:
- net GND: track 35.2 -> 36.3 mm, vias 17 -> 52
- net /power_usb/USB_M-: track 3.85 -> 4.75 mm
- net /power_usb/USB_M+: track 3.83 -> 4.73 mm
- net /connectors_gpios_2_5_4/PA13: track 27.9 -> 28.4 mm
Other:
- board text added: "5V"
- board text added: "CLK"
- board text added: "DIO"
- board text added: "NRST"
- board text added: "PA0"
- board text added: "PA1"
- board text added: "PA12"
- board text added: "PA13"
- board text added: "PA14"
- board text added: "PA15"
- board text added: "PA2"
- board text added: "PB3"
- board text added: "PB4"
- board text added: "PB6"
- board text added: "PB7"
- board text added: "PC14"
- board text added: "PC15"
- board text added: "PH3"

Commit message: final closing part 1
Routing:
- net /connectors_gpios_2_5_4/PB1: track 39.2 -> 26.0 mm
- net /connectors_gpios_2_5_4/PA11: track 37.5 -> 41.6 mm
- net /connectors_gpios_2_5_4/PA4: track 17.4 -> 15.7 mm, vias 1 -> 0
- net GND: track 36.3 -> 37.2 mm, vias 52 -> 57
- net /connectors_gpios_2_5_4/PA3: track 19.7 -> 20.5 mm, vias 1 -> 0
- net /connectors_gpios_2_5_4/PA1: track 25.0 -> 24.4 mm
- net /connectors_gpios_2_5_4/PA6: track 13.3 -> 12.7 mm, vias 1 -> 0
- net /connectors_gpios_2_5_4/PA5: track 15.4 -> 14.9 mm, vias 1 -> 0
- net /connectors_gpios_2_5_4/PB0: track 9.77 -> 10.2 mm, vias 1 -> 0
- net /connectors_gpios_2_5_4/PA13: track 28.4 -> 28.6 mm, vias 0 -> 1
- net /connectors_gpios_2_5_4/PA14: track 30.6 -> 30.5 mm, vias 2 -> 1
- net /connectors_gpios_2_5_4/PA9: track 10.3 -> 10.2 mm, vias 1 -> 0
- net /connectors_gpios_2_5_4/PA7: track 11.5 -> 11.6 mm, vias 1 -> 0
- net /connectors_gpios_2_5_4/PA8: track 8.99 -> 8.96 mm, vias 1 -> 0
Other:
- outline, holes or cut-outs redrawn

Commit message: final closing part 2 no logo
Parts:
- added R7: 10K, Resistor_SMD:R_0603_1608Metric, F.Cu at (148.1, 93.0)
- added R8: 0ohm, Resistor_SMD:R_0603_1608Metric, F.Cu at (155.8, 110.2)
- R2: value 1K -> 0ohm
- R5: value 10K -> 0ohm
- R6: value 0ohm -> 1K
- moved R3 35.5 mm to (156.2, 122.5)
- moved R4 32.5 mm to (156.2, 121.0)
- moved R6 21.7 mm to (153.4, 88.6)
- moved R5 6.03 mm to (153.4, 90.1), turned to 180 degrees
- moved R2 4.25 mm to (156.2, 125.5)
- moved D2 3.02 mm to (153.4, 87.1)
- moved R1 1.26 mm to (156.2, 124.0), turned to 0 degrees
- moved D1 0.25 mm to (156.2, 119.5)
Connections:
- J1 pad 4: unconnected-(J1-ID-Pad4) -> Net-(J1-ID)
- R1 pad 1: +3V3 -> Net-(J1-ID)
- R1 pad 2: Net-(R1-Pad2) -> GND
- R2 pad 1: Net-(R1-Pad2) -> Net-(J1-ID)
- R2 pad 2: Net-(D1-A) -> /connectors_gpios_2_5_4/PA4
- R3 pad 1: /connectors_gpios_2_5_4/PB1 -> +3V3
- R4 pad 2: Net-(D2-A) -> Net-(D1-A)
- R5 pad 1: /connectors_gpios_2_5_4/PH3(BOOT0) -> /connectors_gpios_2_5_4/PB1
- R5 pad 2: GND -> Net-(R5-Pad2)
- R6 pad 1: /connectors_gpios_2_5_4/PA1 -> Net-(R5-Pad2)
- R6 pad 2: Net-(C11-Pad1) -> Net-(D2-A)
Routing:
- net /connectors_gpios_2_5_4/PA4: track 15.7 -> 29.5 mm, vias 0 -> 1
- net Net-(J1-ID): track 0.00 -> 7.62 mm
- net /connectors_gpios_2_5_4/PB1: track 26.0 -> 22.0 mm
- net GND: track 37.2 -> 39.2 mm, vias 57 -> 63
- net Net-(R5-Pad2): track 0.00 -> 1.50 mm
- net Net-(R1-Pad2): track 1.50 -> 0.00 mm
- net +5V_USB: track 21.9 -> 23.2 mm
- net +3V3: track 17.9 -> 18.5 mm

Commit message: production file 1
Parts:
- added G***: LOGO, demo:logo_1_4, B.Cu at (150.0, 78.4)
Other:
- board text added: "stm32L432KCU6_EVAL"

Commit message: production file 1 after review
Parts:
- added G***: LOGO, demo:logo_1_4, F.Cu at (154.4, 105.8)
Routing:
- net +3V3: track 18.5 -> 24.8 mm, vias 7 -> 9
- net GND: track 39.2 -> 42.8 mm
