File: stm32l432kcu6_eval/stm32l432kcu6_eval.kicad_pcb (KiCad board)
At the start: 4 copper layers, 27.4 x 53 mm, 37 parts, among them J1 USB_B_Micro, J2 Conn_01x20_Pin, J3 Conn_01x20_Pin, J4 Conn_01x04_Pin, U1 USBLC6-2SC6, U2 XC6206PxxxMR, U3 STM32L432KCUx, Y1 ASFL1-40.000MHZ-EC-T, Y2 FC-135_32.7680KA-A3_12_5_pF

Commit message: production file 1 final revisio
Parts:
- moved G*** 0.81 mm to (154.5, 105.0)
Connections:
- U3 pad 31: /connectors_gpios_2_5_4/PH3(BOOT) -> /connectors_gpios_2_5_4/PH3(BOOT0)
Routing:
- net /connectors_gpios_2_5_4/PH3(BOOT0): track 15.0 -> 24.7 mm
- net GND: track 42.8 -> 42.9 mm, vias 63 -> 64

Commit message: production file 1 final revision with vias checked
Other:
- board text added: "https://github.com/hedfd434"
Changed lines of the file:
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@@
 	(generator_version "8.0")
 	(general
-		(thickness 1.6)
+		(thickness 1.6062)
 		(legacy_teardrops no)
 	)
@@
 			(layer "dielectric 1"
 				(type "prepreg")
-				(thickness 0.1)
+				(thickness 0.2104)
 				(material "FR4")
 				(epsilon_r 4.5)
@@
 			(layer "In1.Cu"
 				(type "copper")
-				(thickness 0.035)
+				(thickness 0.0152)
 			)
 			(layer "dielectric 2"
 				(type "core")
-				(thickness 1.24)
+				(thickness 1.065)
 				(material "FR4")
 				(epsilon_r 4.5)
@@
 			(layer "In2.Cu"
 				(type "copper")
-				(thickness 0.035)
+				(thickness 0.0152)
 			)
 			(layer "dielectric 3"
 				(type "prepreg")
-				(thickness 0.1)
+				(thickness 0.2104)
 				(material "FR4")
 				(epsilon_r 4.5)
@@
 	)
 	(gr_line
+		(start 144.2 100)
+		(end 144.2 99.5)
+		(stroke
+			(width 0.1)
+			(type default)
+		)
+		(layer "User.2")
+	)
+	(gr_line
 		(start 161.43 88.57)
 		(end 161.43 91.11)
@@
 	)
 	(gr_line
+		(start 155.8 100)
+		(end 155.8 99.5)
+		(stroke
+			(width 0.1)
+			(type default)
+		)
+		(layer "User.2")
+	)
+	(gr_line
 		(start 138.57 86.03)
 		(end 138.57 88.57)
@@
 	)
 	(gr_line
+		(start 150 100)
+		(end 144.2 100)
+		(stroke
+			(width 0.1)
+			(type default)
+		)
+		(layer "User.2")
+	)
+	(gr_line
 		(start 161.43 83.49)
 		(end 161.43 86.03)
@@
 		(layer "User.2")
 	)
+	(gr_text "https://github.com/hedfd434"
+		(at 144.2 99.5 -90)
+		(layer "B.SilkS")
+		(effects
+			(font
+				(size 1 1)
+				(thickness 0.15)
+			)
+			(justify mirror)
+		)
+	)
 	(gr_text "stm32L432KCU6_EVAL"
-		(at 155.715 100 270)
+		(at 155.8 100 270)
 		(layer "B.SilkS")
 		(effects
