File: stm32l432kcu6_eval/stm32l432kcu6_eval.kicad_sch (KiCad schematic)
At the start: 0 parts

Commit message: board save 1
Other:
- sheet mcu_osccillators ports: added MCU_USB_DM, MCU_USB_DP, MCU_USB_NOE; removed none
Changed lines of the file:
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@@
+			)
+		)
+		(pin "MCU_USB_DM" bidirectional
+			(at 213.36 99.06 0)
+			(effects
+				(font
+					(size 1.27 1.27)
+				)
+				(justify right)
+			)
+		)
+		(pin "MCU_USB_DP" bidirectional
+			(at 213.36 95.25 0)
+			(effects
+				(font
+					(size 1.27 1.27)
+				)
+				(justify right)
+			)
+		)
+		(pin "MCU_USB_NOE" bidirectional
+			(at 213.36 91.44 0)
+			(effects
+				(font
+					(size 1.27 1.27)
+				)
+				(justify right)
 			)
 		)

Commit message: board save 4
Other:
- sheet connectors_gpios_2_5_4 ports: added PAX(BUS), SWCLK, SWDIO; removed none
- sheet mcu_osccillators ports: added PAX(BUS), SWCLK, SWDIO; removed MCU_USB_DM, MCU_USB_DP, MCU_USB_NOE
Changed lines of the file:
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@@
 	(generator_version "8.0")
 	(paper "A4")
+	(wire
+		(pts
+			(xy 196.85 138.43) (xy 196.85 111.76)
+		)
+		(stroke
+			(width 0)
+			(type default)
+		)
+	)
+	(wire
+		(pts
+			(xy 248.92 99.06) (xy 248.92 123.19)
+		)
+		(stroke
+			(width 0)
+			(type default)
+		)
+	)
+	(wire
+		(pts
+			(xy 203.2 129.54) (xy 203.2 111.76)
+		)
+		(stroke
+			(width 0)
+			(type default)
+		)
+	)
+	(wire
+		(pts
+			(xy 237.49 138.43) (xy 196.85 138.43)
+		)
+		(stroke
+			(width 0)
+			(type default)
+		)
+	)
+	(wire
+		(pts
+			(xy 213.36 99.06) (xy 248.92 99.06)
+		)
+		(stroke
+			(width 0)
+			(type default)
+		)
+	)
+	(wire
+		(pts
+			(xy 237.49 129.54) (xy 203.2 129.54)
+		)
+		(stroke
+			(width 0)
+			(type default)
+		)
+	)
 	(sheet
-		(at 181.61 132.08)
+		(at 226.06 71.12)
 		(size 29.21 17.78)
 		(fields_autoplaced yes)
@@
 		)
 		(property "Sheetname" "power_usb"
-			(at 181.61 131.3684 0)
+			(at 226.06 70.4084 0)
 			(effects
 				(font
@@
 		)
 		(property "Sheetfile" "untitled.kicad_sch"
-			(at 181.61 150.4446 0)
+			(at 226.06 89.4846 0)
 			(effects
 				(font
@@
 			)
 		)
-		(pin "MCU_USB_DM" bidirectional
+		(pin "SWDIO" bidirectional
+			(at 196.85 111.76 270)
+			(effects
+				(font
+					(size 1.27 1.27)
+				)
+				(justify left)
+			)
+		)
+		(pin "SWCLK" bidirectional
+			(at 203.2 111.76 270)
+			(effects
+				(font
+					(size 1.27 1.27)
+				)
+				(justify left)
+			)
+		)
+		(pin "PAX(BUS)" bidirectional
 			(at 213.36 99.06 0)
-			(effects
-				(font
-					(size 1.27 1.27)
-				)
-				(justify right)
-			)
-		)
-		(pin "MCU_USB_DP" bidirectional
-			(at 213.36 95.25 0)
-			(effects
-				(font
-					(size 1.27 1.27)
-				)
-				(justify right)
-			)
-		)
-		(pin "MCU_USB_NOE" bidirectional
-			(at 213.36 91.44 0)
 			(effects
 				(font
@@
 			)
 		)
+		(pin "SWCLK" bidirectional
+			(at 237.49 129.54 180)
+			(effects
+				(font
+					(size 1.27 1.27)
+				)
+				(justify left)
+			)
+		)
+		(pin "SWDIO" bidirectional
+			(at 237.49 138.43 180)
+			(effects
+				(font
+					(size 1.27 1.27)
+				)
+				(justify left)
+			)
+		)
+		(pin "PAX(BUS)" bidirectional
+			(at 248.92 123.19 90)
+			(effects
+				(font
+					(size 1.27 1.27)
+				)
+				(justify right)
+			)
+		)

Commit message: pin arragment 1
Other:
- sheet connectors_gpios_2_5_4 ports: added PBX(BUS), PHCNX; removed none
- sheet mcu_osccillators ports: added PBX(BUS), PHCNX; removed none
- sheet power_usb ports: added PAX(BUS); removed none
Changed lines of the file:
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@@
 	(generator_version "8.0")
 	(paper "A4")
-	(wire
-		(pts
-			(xy 196.85 138.43) (xy 196.85 111.76)
-		)
-		(stroke
-			(width 0)
-			(type default)
-		)
-	)
-	(wire
-		(pts
-			(xy 248.92 99.06) (xy 248.92 123.19)
-		)
-		(stroke
-			(width 0)
-			(type default)
-		)
-	)
-	(wire
-		(pts
-			(xy 203.2 129.54) (xy 203.2 111.76)
-		)
-		(stroke
-			(width 0)
-			(type default)
-		)
-	)
-	(wire
-		(pts
-			(xy 237.49 138.43) (xy 196.85 138.43)
-		)
-		(stroke
-			(width 0)
-			(type default)
-		)
-	)
-	(wire
-		(pts
-			(xy 213.36 99.06) (xy 248.92 99.06)
-		)
-		(stroke
-			(width 0)
-			(type default)
-		)
-	)
-	(wire
-		(pts
-			(xy 237.49 129.54) (xy 203.2 129.54)
+	(junction
+		(at 154.94 95.25)
+		(diameter 0)
+		(color 0 0 0 0)
+	)
+	(wire
+		(pts
+			(xy 116.84 134.62) (xy 116.84 107.95)
+		)
+		(stroke
+			(width 0)
+			(type default)
+		)
+	)
+	(wire
+		(pts
+			(xy 185.42 95.25) (xy 185.42 119.38)
+		)
+		(stroke
+			(width 0)
+			(type default)
+		)
+	)
+	(wire
+		(pts
+			(xy 179.07 119.38) (xy 179.07 99.06)
+		)
+		(stroke
+			(width 0)
+			(type default)
+		)
+	)
+	(wire
+		(pts
+			(xy 120.65 125.73) (xy 120.65 107.95)
+		)
+		(stroke
+			(width 0)
+			(type default)
+		)
+	)
+	(wire
+		(pts
+			(xy 154.94 95.25) (xy 154.94 85.09)
+		)
+		(stroke
+			(width 0)
+			(type default)
+		)
+	)
+	(wire
+		(pts
+			(xy 162.56 134.62) (xy 116.84 134.62)
+		)
+		(stroke
+			(width 0)
+			(type default)
+		)
+	)
+	(wire
+		(pts
+			(xy 138.43 95.25) (xy 154.94 95.25)
+		)
+		(stroke
+			(width 0)
+			(type default)
+		)
+	)
+	(wire
+		(pts
+			(xy 172.72 119.38) (xy 172.72 102.87)
+		)
+		(stroke
+			(width 0)
+			(type default)
+		)
+	)
+	(wire
+		(pts
+			(xy 179.07 99.06) (xy 138.43 99.06)
+		)
+		(stroke
+			(width 0)
+			(type default)
+		)
+	)
+	(wire
+		(pts
+			(xy 162.56 125.73) (xy 120.65 125.73)
+		)
+		(stroke
+			(width 0)
+			(type default)
+		)
+	)
+	(wire
+		(pts
+			(xy 172.72 102.87) (xy 138.43 102.87)
+		)
+		(stroke
+			(width 0)
+			(type default)
+		)
+	)
+	(wire
+		(pts
+			(xy 154.94 95.25) (xy 185.42 95.25)
 		)
 		(stroke
@@
 	)
 	(sheet
-		(at 226.06 71.12)
+		(at 151.13 67.31)
 		(size 29.21 17.78)
 		(fields_autoplaced yes)
@@
 		)
 		(property "Sheetname" "power_usb"
-			(at 226.06 70.4084 0)
+			(at 151.13 66.5984 0)
 			(effects
 				(font
@@
 		)
 		(property "Sheetfile" "untitled.kicad_sch"
-			(at 226.06 89.4846 0)
+			(at 151.13 85.6746 0)
 			(effects
 				(font
@@
 				)
 				(justify left top)
+			)
+		)
+		(pin "PAX(BUS)" bidirectional
+			(at 154.94 85.09 270)
+			(effects
+				(font
+					(size 1.27 1.27)
+				)
+				(justify left)
 			)
 		)
@@
 	)
 	(sheet
-		(at 187.96 85.09)
+		(at 113.03 81.28)
 		(size 25.4 26.67)
 		(fields_autoplaced yes)
@@
 		)
 		(property "Sheetname" "mcu_osccillators"
-			(at 187.96 84.3784 0)
+			(at 113.03 80.5684 0)
 			(effects
 				(font
@@
 		)
 		(property "Sheetfile" "mcu_osccillators.kicad_sch"
-			(at 187.96 112.3446 0)
+			(at 113.03 108.5346 0)
 			(effects
 				(font
@@
 		)
 		(pin "SWDIO" bidirectional
-			(at 196.85 111.76 270)
+			(at 116.84 107.95 270)
 			(effects
 				(font
@@
 		)
 		(pin "SWCLK" bidirectional
-			(at 203.2 111.76 270)
+			(at 120.65 107.95 270)
 			(effects
 				(font
@@
 		)
 		(pin "PAX(BUS)" bidirectional
-			(at 213.36 99.06 0)
+			(at 138.43 95.25 0)
+			(effects
+				(font
+					(size 1.27 1.27)
+				)
+				(justify right)
+			)
+		)
+		(pin "PHCNX" bidirectional
+			(at 138.43 99.06 0)
+			(effects
+				(font
+					(size 1.27 1.27)
+				)
+				(justify right)
+			)
+		)
+		(pin "PBX(BUS)" bidirectional
+			(at 138.43 102.87 0)
 			(effects
 				(font
@@
 	)
 	(sheet
-		(at 237.49 123.19)
+		(at 162.56 119.38)
 		(size 29.21 24.13)
 		(fields_autoplaced yes)
@@
 		)
 		(property "Sheetname" "connectors_gpios_2_5_4"
-			(at 237.49 122.4784 0)
+			(at 162.56 118.6684 0)
 			(effects
 				(font
@@
 		)
 		(property "Sheetfile" "connectors_gpios_2_5_4.kicad_sch"
-			(at 237.49 147.9046 0)
+			(at 162.56 144.0946 0)
 			(effects
 				(font
@@
 		)
 		(pin "SWCLK" bidirectional
-			(at 237.49 129.54 180)
+			(at 162.56 125.73 180)
 			(effects
 				(font
@@
 		)
 		(pin "SWDIO" bidirectional
-			(at 237.49 138.43 180)
+			(at 162.56 134.62 180)
 			(effects
 				(font
@@
 		)
 		(pin "PAX(BUS)" bidirectional
-			(at 248.92 123.19 90)
-			(effects
-				(font
+			(at 185.42 119.38 90)
+			(effects
+				(font
+					(size 1.27 1.27)
+				)
+				(justify right)
+			)
+		)
+		(pin "PBX(BUS)" bidirectional
+			(at 172.72 119.38 90)
+			(effects
+				(font
+					(size 1.27 1.27)
+				)
+				(justify right)
+			)
+		)
+		(pin "PHCNX" bidirectional
+			(at 179.07 119.38 90)
+			(effects
+				(font
