File: stm32l432kcu6_eval/_autosave-stm32l432kcu6_eval.kicad_pcb (KiCad board)
At the start: 4 copper layers, 27.4 x 53 mm, 33 parts, among them J1 Conn_01x04_Pin, J2 Conn_01x20_Pin, J4 Conn_01x20_Pin, J5 USB_B_Micro, U1 STM32L432KCUx, U2 XC6206PxxxMR, U3 USBLC6-2SC6, Y1 ASFL1-40.000MHZ-EC-T, Y2 FC-135_32.7680KA-A3_12_5_pF

Commit message: organisation save 1
Parts:
- moved C11 24.3 mm to (173.7, 112.7)
- moved C4 21.2 mm to (165.8, 92.0)
- moved R1 18.6 mm to (167.2, 96.4)
- moved R6 18.5 mm to (173.9, 114.7)
- moved C10 11.7 mm to (186.8, 97.5)
- moved C5 9.50 mm to (186.6, 99.7)
- moved S1 6.29 mm to (124.9, 88.3)
- moved S3 2.24 mm to (169.4, 112.9)
Changed lines of the file:
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@@
 	(footprint "custom_part_library_1:B3U1000PM_3D_MODEL"
 		(layer "F.Cu")
-		(at 168.7 110.775 90)
+		(at 169.4 112.9 90)
 		(descr "B3U-1000PM-3")
 		(tags "Switch")
@@
 	(footprint "Capacitor_SMD:C_0603_1608Metric"
 		(layer "F.Cu")
-		(at 192.125 96.9)
+		(at 173.7 112.7)
 		(descr "Capacitor SMD 0603 (1608 Metric), square (rectangular) end terminal, IPC_7351 nominal, (Body size source: IPC-SM-782 page 76, https://www.pcb-3d.com/wordpress/wp-content/uploads/ipc-sm-782a_amendment_1_and_2.pdf), generated with kicad-footprint-generator")
 		(tags "capacitor")
@@
 	(footprint "Resistor_SMD:R_0603_1608Metric"
 		(layer "F.Cu")
-		(at 178.725 111)
+		(at 167.225 96.4)
 		(descr "Resistor SMD 0603 (1608 Metric), square (rectangular) end terminal, IPC_7351 nominal, (Body size source: IPC-SM-782 page 72, https://www.pcb-3d.com/wordpress/wp-content/uploads/ipc-sm-782a_amendment_1_and_2.pdf), generated with kicad-footprint-generator")
 		(tags "resistor")
@@
 	(footprint "Capacitor_SMD:C_0603_1608Metric"
 		(layer "F.Cu")
-		(at 175.8 110.775 90)
+		(at 165.8 92.025 90)
 		(descr "Capacitor SMD 0603 (1608 Metric), square (rectangular) end terminal, IPC_7351 nominal, (Body size source: IPC-SM-782 page 76, https://www.pcb-3d.com/wordpress/wp-content/uploads/ipc-sm-782a_amendment_1_and_2.pdf), generated with kicad-footprint-generator")
 		(tags "capacitor")
@@
 	(footprint "Capacitor_SMD:C_0603_1608Metric"
 		(layer "F.Cu")
-		(at 186.8 90.2)
+		(at 186.6 99.7)
 		(descr "Capacitor SMD 0603 (1608 Metric), square (rectangular) end terminal, IPC_7351 nominal, (Body size source: IPC-SM-782 page 76, https://www.pcb-3d.com/wordpress/wp-content/uploads/ipc-sm-782a_amendment_1_and_2.pdf), generated with kicad-footprint-generator")
 		(tags "capacitor")
@@
 	(footprint "Resistor_SMD:R_0603_1608Metric"
 		(layer "F.Cu")
-		(at 186.8 101.5)
+		(at 173.9 114.7)
 		(descr "Resistor SMD 0603 (1608 Metric), square (rectangular) end terminal, IPC_7351 nominal, (Body size source: IPC-SM-782 page 72, https://www.pcb-3d.com/wordpress/wp-content/uploads/ipc-sm-782a_amendment_1_and_2.pdf), generated with kicad-footprint-generator")
 		(tags "resistor")
@@
 	(footprint "custom_part_library_1:B3U1000PM_3D_MODEL"
 		(layer "F.Cu")
-		(at 129.297918 92.802082)
+		(at 124.9 88.3)
 		(descr "B3U-1000PM-3")
 		(tags "Switch")
@@
 	(footprint "Capacitor_SMD:C_0603_1608Metric"
 		(layer "F.Cu")
-		(at 194.775 89)
+		(at 186.8 97.5)
 		(descr "Capacitor SMD 0603 (1608 Metric), square (rectangular) end terminal, IPC_7351 nominal, (Body size source: IPC-SM-782 page 76, https://www.pcb-3d.com/wordpress/wp-content/uploads/ipc-sm-782a_amendment_1_and_2.pdf), generated with kicad-footprint-generator")
 		(tags "capacitor")
