File: stm32l432kcu6_eval/connectors_gpios_2_5_4.kicad_sch (KiCad schematic)
At the start: 2 parts, among them J1 Conn_01x04_Pin, J2 Conn_01x04_Pin

Commit message: board save 4
Parts:
- removed J2: Conn_01x04_Pin, Connector_PinSocket_2.54mm:PinSocket_1x04_P2.54mm_Horizontal, symbol Connector:Conn_01x04_Pin
- added J2, J4: Conn_01x20_Pin, Connector_PinSocket_2.54mm:PinSocket_1x20_P2.54mm_Vertical, symbol Connector:Conn_01x20_Pin
Connections:
- net +3V3: now reaches J1.1 (Pin_1)
- net PA13: now reaches J1.2 (Pin_2)
- net PA13: now also J2.14 (Pin_14)
- net PA14: now reaches J1.3 (Pin_3)
- net PA14: now also J2.15 (Pin_15)
- net GND: now reaches J1.4 (Pin_4)
- new net NRST: J4.8 (Pin_8)
- new net PA0: J2.1 (Pin_1)
- new net PA1: J2.2 (Pin_2)
- new net PA10: J2.11 (Pin_11)
- new net PA11: J2.12 (Pin_12)
- new net PA12: J2.13 (Pin_13)
- new net PA15: J2.16 (Pin_16)
- new net PA2: J2.3 (Pin_3)
- new net PA3: J2.4 (Pin_4)
- new net PA4: J2.5 (Pin_5)
- new net PA5: J2.6 (Pin_6)
- new net PA6: J2.7 (Pin_7)
- new net PA7: J2.8 (Pin_8)
- new net PA8: J2.9 (Pin_9)
- new net PA9: J2.10 (Pin_10)
- new net PB0: J4.1 (Pin_1)
- new net PB1: J4.2 (Pin_2)
- new net PB3: J4.3 (Pin_3)
- new net PB4: J4.4 (Pin_4)
- new net PB5: J4.5 (Pin_5)
- new net PB6: J4.6 (Pin_6)
- new net PB7: J4.7 (Pin_7)
- new net PC14(OSC_IN): J4.10 (Pin_10), J4.11 (Pin_11)
- new net PH3(BOOT): J4.9 (Pin_9)
Other:
- moved on the sheet: J1

Commit message: pin arragment 1
Parts:
- added C10, C11, C4: 100nF, Capacitor_SMD:C_0603_1608Metric, symbol Device:C_Small
- added D1, D2: LED, LED_SMD:LED_0603_1608Metric, symbol Device:LED
- added R1: 10K, Resistor_SMD:R_0603_1608Metric, symbol Device:R_Small
- added R2, R3, R4, R5, R6: R_Small, Resistor_SMD:R_0603_1608Metric, symbol Device:R_Small
- added S1, S2, S3: B3U-1000PM, custom_part_library_1:B3U1000PM_3D_MODEL, symbol B3U-1000PM_OMRON:B3U-1000PM
Connections:
- net +3V3: now also R4.1, S2.1
- net GND: now also C10.2, C11.2, C4.2, D1.1 (K), D2.1 (K), R1.2, S1.1, S3.1
- net NRST: now also J2.13 (Pin_13), C10.1, S1.2; no longer J4.8 (Pin_8)
- net PA0: now also J2.14 (Pin_14); no longer J2.1 (Pin_1)
- net PA1: now also J2.15 (Pin_15), R6.1; no longer J2.2 (Pin_2)
- net PA10: now also J4.13 (Pin_13); no longer J2.11 (Pin_11)
- net PA11: now also J4.14 (Pin_14); no longer J2.12 (Pin_12)
- net PA12: now also J4.15 (Pin_15); no longer J2.13 (Pin_13)
- net PA13: now also J4.16 (Pin_16); no longer J2.14 (Pin_14)
- net PA14: now also J4.17 (Pin_17); no longer J2.15 (Pin_15)
- net PA15: now also J2.4 (Pin_4); no longer J2.16 (Pin_16)
- net PA2: now also J2.16 (Pin_16); no longer J2.3 (Pin_3)
- net PA3: now also J4.6 (Pin_6); no longer J2.4 (Pin_4)
- net PA4: now also J4.7 (Pin_7); no longer J2.5 (Pin_5)
- net PA5: now also J4.8 (Pin_8); no longer J2.6 (Pin_6)
- net PA6: now also J4.9 (Pin_9); no longer J2.7 (Pin_7)
- net PA7: now also J4.10 (Pin_10); no longer J2.8 (Pin_8)
- net PA8: now also J4.11 (Pin_11); no longer J2.9 (Pin_9)
- net PA9: now also J4.12 (Pin_12); no longer J2.10 (Pin_10)
- net PB0: no longer J4.1 (Pin_1)
- net PB1: now also R5.1; no longer J4.2 (Pin_2)
- net PB3: now also J2.5 (Pin_5); no longer J4.3 (Pin_3)
- net PB4: now also J2.6 (Pin_6); no longer J4.4 (Pin_4)
- net PB5: now also J2.7 (Pin_7); no longer J4.5 (Pin_5)
- net PB6: now also J2.8 (Pin_8); no longer J4.6 (Pin_6)
- net PB7: now also J2.9 (Pin_9); no longer J4.7 (Pin_7)
- net PC14(OSC_IN): now also J2.11 (Pin_11); no longer J4.10 (Pin_10), J4.11 (Pin_11)
- net PH3(BOOT): now also J2.10 (Pin_10); no longer J4.9 (Pin_9)
- new net: R3.1, R5.2
- new net: D2.2 (A), R3.2
- new net: R2.1, R4.2
- new net: C11.1, R6.2, S3.2
- new net: D1.2 (A), R2.2
- new net PC15(OSC_OUT): J2.12 (Pin_12)
- new net PH3(BOOT0): C4.1, R1.1, S2.2
- no-connect marks 0 -> 1

Commit message: organisation save 1
Parts:
- J1: footprint Connector_PinSocket_2.54mm:PinSocket_1x04_P2.54mm_Horizontal -> Connector_PinHeader_2.54mm:PinHeader_1x04_P2.54mm_Horizontal
- J2, J4: footprint Connector_PinSocket_2.54mm:PinSocket_1x20_P2.54mm_Vertical -> Connector_PinHeader_2.54mm:PinHeader_1x20_P2.54mm_Vertical
Connections:
- net +3V3: now also J1.4 (Pin_4); no longer J1.1 (Pin_1)
- net GND: now also J1.1 (Pin_1); no longer J1.4 (Pin_4)
- net PA13: now also J1.3 (Pin_3); no longer J1.2 (Pin_2)
- net PA14: now also J1.2 (Pin_2); no longer J1.3 (Pin_3)
- net PA3: now also J4.4 (Pin_4); no longer J4.6 (Pin_6)
- net PA4: now also J4.5 (Pin_5); no longer J4.7 (Pin_7)
- net PA5: now also J4.6 (Pin_6); no longer J4.8 (Pin_8)
- net PA6: now also J4.7 (Pin_7); no longer J4.9 (Pin_9)
- net PA7: now also J4.8 (Pin_8); no longer J4.10 (Pin_10)
- net PB0: now also J4.9 (Pin_9)
- net PB1: now also J4.10 (Pin_10)
