File: stm32l432kcu6_eval/connectors_gpios_2_5_4.kicad_sch (KiCad schematic)
At the start: 17 parts, among them J1 Conn_01x04_Pin, J2 Conn_01x20_Pin, J4 Conn_01x20_Pin

Commit message: organisation save 2
Parts:
- R1: renamed from R4; value R_Small -> 0ohm
- R2: value R_Small -> 1K
- R3: renamed from R5; value R_Small -> 0ohm
- R4: renamed from R3; value R_Small -> 1K
- R6: value R_Small -> 0ohm
- renumbered C4 to C10, C10 to C9, J4 to J3, J1 to J4, R1 to R5
Connections:
- no-connect marks 1 -> 0
Other:
- moved on the sheet: C10, C11, C9, D1, D2, J2, J3, J4, R1, R2, R3, R4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

Commit message: project final works save 1
Connections:
- net PA13: now also J4.2 (Pin_2); no longer J4.3 (Pin_3)
- net PA14: now also J4.3 (Pin_3); no longer J4.2 (Pin_2)
- net PH3(BOOT): no longer J2.10 (Pin_10)
- net PH3(BOOT0): now also J2.10 (Pin_10)

Commit message: project final works save 2
Connections:
- net +3V3: now also J2.1 (Pin_1), J2.18 (Pin_18), J2.2 (Pin_2), J3.1 (Pin_1), J3.20 (Pin_20)
- net GND: now also J2.17 (Pin_17), J2.3 (Pin_3), J3.18 (Pin_18), J3.19 (Pin_19), J3.2 (Pin_2), J3.3 (Pin_3)
- net +5V_USB: now reaches J2.19 (Pin_19)
- net +5V_USB: now also J2.20 (Pin_20)

Commit message: project final works save 3
Connections:
- net PA13: now also J4.3 (Pin_3); no longer J4.2 (Pin_2)
- net PA14: now also J4.2 (Pin_2); no longer J4.3 (Pin_3)
Changed lines of the file:
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@@
 	)
 	(label "SWCLK"
-		(at 49.53 121.92 0)
+		(at 49.53 119.38 0)
 		(fields_autoplaced yes)
 		(effects
@@
 	)
 	(label "SWDIO"
-		(at 49.53 119.38 0)
-		(fields_autoplaced yes)
-		(effects
+		(at 49.53 121.92 0)
+		(fields_autoplaced yes)
+		(effects

Commit message: final closing part 2 no logo
Parts:
- renumbered R1 to R3, R2 to R4, R3 to R5, R4 to R6, R5 to R7, R6 to R8
Changed lines of the file:
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@@
 		(dnp no)
 		(fields_autoplaced yes)
-		(property "Reference" "R4"
+		(property "Reference" "R6"
 			(at 123.19 121.92 90)
 			(effects
@@
 			(project "stm32l432kcu6_eval"
 				(path "/8c9f4ed2-db3b-402c-9437-65e91cdde455/d780161e-b7fd-448c-b7ed-1aa3165a374c"
-					(reference "R4")
+					(reference "R6")
 					(unit 1)
 				)
@@
 		(dnp no)
 		(fields_autoplaced yes)
-		(property "Reference" "R1"
+		(property "Reference" "R3"
 			(at 114.3 111.76 90)
 			(effects
@@
 			(project "stm32l432kcu6_eval"
 				(path "/8c9f4ed2-db3b-402c-9437-65e91cdde455/d780161e-b7fd-448c-b7ed-1aa3165a374c"
-					(reference "R1")
+					(reference "R3")
 					(unit 1)
 				)
@@
 		(dnp no)
 		(fields_autoplaced yes)
-		(property "Reference" "R5"
+		(property "Reference" "R7"
 			(at 237.49 120.6499 0)
 			(effects
@@
 			(project "stm32l432kcu6_eval"
 				(path "/8c9f4ed2-db3b-402c-9437-65e91cdde455/d780161e-b7fd-448c-b7ed-1aa3165a374c"
-					(reference "R5")
+					(reference "R7")
 					(unit 1)
 				)
@@
 		(dnp no)
 		(fields_autoplaced yes)
-		(property "Reference" "R6"
+		(property "Reference" "R8"
 			(at 57.15 165.1 90)
 			(effects
@@
 			(project "stm32l432kcu6_eval"
 				(path "/8c9f4ed2-db3b-402c-9437-65e91cdde455/d780161e-b7fd-448c-b7ed-1aa3165a374c"
-					(reference "R6")
+					(reference "R8")
 					(unit 1)
 				)
@@
 		(dnp no)
 		(fields_autoplaced yes)
-		(property "Reference" "R3"
+		(property "Reference" "R5"
 			(at 114.3 121.92 90)
 			(effects
@@
 			(project "stm32l432kcu6_eval"
 				(path "/8c9f4ed2-db3b-402c-9437-65e91cdde455/d780161e-b7fd-448c-b7ed-1aa3165a374c"
-					(reference "R3")
+					(reference "R5")
 					(unit 1)
 				)
@@
 		(dnp no)
 		(fields_autoplaced yes)
-		(property "Reference" "R2"
+		(property "Reference" "R4"
 			(at 123.19 111.76 90)
 			(effects
@@
 			(project ""
 				(path "/8c9f4ed2-db3b-402c-9437-65e91cdde455/d780161e-b7fd-448c-b7ed-1aa3165a374c"
-					(reference "R2")
-					(unit 1)
-				)
+					(reference "R4")
+					(unit 1)
+				)
