File: stm32l432kcu6_eval/untitled.kicad_sch (KiCad schematic)
At the start: 7 parts, among them J3 USB_C_Receptacle, U2 XC6206PxxxMR, U3 USBLC6-2SC6

Commit message: board save 1
Parts:
- C3, C5: value C_Small -> 100nF
- FB1: value FerriteBead_Small -> value
Connections:
- net +5V_USB: now reaches F1.1
- net +5V_USB: now also J3.A4 (VBUS), J3.A9 (VBUS), J3.B4 (VBUS), J3.B9 (VBUS), U3.5 (VBUS)
- net at F1.2: now also FB1.1
- net +3V3: now reaches C5.1
- net +3V3: now also U2.2 (VO)
- net GND: now reaches C5.2
- net GND: now also C3.2, J3.A1 (GND), J3.A12 (GND), J3.B1 (GND), J3.B12 (GND), J3.S1 (SHIELD), U2.1 (GND), U3.2 (GND)
- net at U2.3 (VI): now also C3.1, FB1.2
- net USB_D-: now reaches U3.1 (I/O1)
- net USB_D-: now also J3.A7 (D-), J3.B7 (D-)
- net USB_D+: now reaches U3.3 (I/O2)
- net USB_D+: now also J3.A6 (D+), J3.B6 (D+)
- net MCU_USB_DP: now reaches U3.4 (I/O2)
- net MCU_USB_DM: now reaches U3.6 (I/O1)
- no-connect marks 0 -> 13
Other:
- moved on the sheet: C3, C5, F1, FB1, U2, U3

Commit message: board save 4
Connections:
- net MCU_USB_DM: now also U3.4 (I/O2); no longer U3.6 (I/O1)
- net MCU_USB_DP: now also U3.6 (I/O1); no longer U3.4 (I/O2)
- net USB_D+: now also U3.1 (I/O1); no longer U3.3 (I/O2)
- net USB_D-: now also U3.3 (I/O2); no longer U3.1 (I/O1)
Changed lines of the file:
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@@
 	(global_label "USB_D+"
 		(shape input)
-		(at 143.51 104.14 180)
+		(at 143.51 99.06 180)
 		(fields_autoplaced yes)
 		(effects
@@
 		)
 		(property "Intersheetrefs" "${INTERSHEET_REFS}"
-			(at 132.9048 104.14 0)
+			(at 132.9048 99.06 0)
 			(effects
 				(font
@@
 	(global_label "USB_D-"
 		(shape input)
-		(at 143.51 99.06 180)
+		(at 143.51 104.14 180)
 		(fields_autoplaced yes)
 		(effects
@@
 		)
 		(property "Intersheetrefs" "${INTERSHEET_REFS}"
-			(at 132.9048 99.06 0)
+			(at 132.9048 104.14 0)
 			(effects
 				(font
@@
 	(hierarchical_label "MCU_USB_DP"
 		(shape bidirectional)
-		(at 161.29 102.87 0)
+		(at 161.29 100.33 0)
 		(fields_autoplaced yes)
 		(effects
@@
 	(hierarchical_label "MCU_USB_DM"
 		(shape bidirectional)
-		(at 161.29 100.33 0)
+		(at 161.29 102.87 0)
 		(fields_autoplaced yes)
 		(effects

Commit message: pin arragment 1
Parts:
- removed J3: USB_C_Receptacle, Connector_USB:USB_C_Receptacle_Molex_105450-0101, symbol Connector:USB_C_Receptacle
- added J5: USB_B_Micro, Connector_USB:USB_Micro-B_Molex-105017-0001, symbol Connector:USB_B_Micro
Connections:
- net +5V_USB: now also J5.1 (VBUS)
- net GND: now also J5.5 (GND), J5.6 (Shield)
- net MCU_USB_DM renamed PA11
- net MCU_USB_DP renamed PA12
- net USB_D+ renamed USB_M+
- net USB_M+: now also J5.3 (D+)
- net USB_D- renamed USB_M-
- net USB_M-: now also J5.2 (D-)
- no-connect marks 13 -> 0
Other:
- moved on the sheet: U3

Commit message: organisation save 1
Other:
- moved on the sheet: C3, C5, F1, FB1, J5, U2, U3

Commit message: organisation save 2
Parts:
- renumbered C3 to C1, C5 to C2, J5 to J1, U3 to U1
Connections:
- net PA11: now also U1.3 (I/O2); no longer U1.4 (I/O2)
- net PA12: now also U1.1 (I/O1); no longer U1.6 (I/O1)
- net USB_M+: now also U1.6 (I/O1); no longer U1.1 (I/O1)
- net USB_M-: now also U1.4 (I/O2); no longer U1.3 (I/O2)
- no-connect marks 0 -> 1
Other:
- moved on the sheet: C1, C2, F1, FB1, U2

Commit message: final closing part 2 no logo
Parts:
- added R1, R2: 0ohm, Resistor_SMD:R_0603_1608Metric, symbol Device:R_Small
Connections:
- net GND: now also R1.2
- net at J1.4 (ID): now also R1.1, R2.1
- new net PA4: R2.2
- no-connect marks 1 -> 0
Other:
- moved on the sheet: C1, C2, F1, FB1, U1, U2
